File: PCBs/Kicad-Files/ESP32_Breakout_Carrier/ESPuino.sch (KiCad schematic (older format))
At the start: 15 parts, among them J1 SD-Card Reader, J2 RFID-RC522, J3 Adafruit MAX98357, J4 Rotary Encode, J5 Next, J6 Prev, J7 Pause, J8 WS2812, J9 Power, Q1 BC337, Q2 IRF9540N, U1 ESP32-DEVKITC-32U

Commit message: KiCad-Files umbenennen: ESP32_Breakout_Carrier
Parts:
- U1: footprint ESP32-DEVKITC-32U:MODULE_ESP32-DEVKITC-32U -> ESP32_Breakout_Carrier:MODULE_ESP32-DEVKITC-32U; symbol Tonuino-ESP32_2-rescue:ESP32-DEVKITC-32U-ESP32-DEVKITC-32U -> ESPuino-rescue:ESP32-DEVKITC-32U-ESP32-DEVKITC-32U
Connections:
- no-connect marks 0 -> 16
Changed lines of the file:
@@
 $EndDescr
 $Comp
-L Tonuino-ESP32_2-rescue:ESP32-DEVKITC-32U-ESP32-DEVKITC-32U U1
+L ESPuino-rescue:ESP32-DEVKITC-32U-ESP32-DEVKITC-32U U1
 U 1 1 5F79096D
 P 8100 2650
 F 0 "U1" H 8100 3817 50  0000 C CNN
 F 1 "ESP32-DEVKITC-32U" H 8100 3726 50  0000 C CNN
-F 2 "ESP32-DEVKITC-32U:MODULE_ESP32-DEVKITC-32U" H 8100 2650 50  0001 L BNN
+F 2 "ESP32_Breakout_Carrier:MODULE_ESP32-DEVKITC-32U" H 8100 2650 50  0001 L BNN
 F 3 "Manufacturer Recommendations" H 8100 2650 50  0001 L BNN
 F 4 "ESPRESSIF" H 8100 2650 50  0001 L BNN "Field4"
@@
 	2750 2300 2750 2650
 Connection ~ 2750 2300
+NoConn ~ 8900 2050
+NoConn ~ 8900 2150
+NoConn ~ 8900 3050
+NoConn ~ 8900 3150
+NoConn ~ 8900 3350
+NoConn ~ 8900 3450
+NoConn ~ 8900 3550
+NoConn ~ 7300 3450
+NoConn ~ 7300 3350
+NoConn ~ 7300 3250
+NoConn ~ 7300 2050
+NoConn ~ 7300 1950
+NoConn ~ 7300 1850
+NoConn ~ 4750 6650
+NoConn ~ 4650 6650
+NoConn ~ 4750 5250
 $EndSCHEMATC
