File: PCBs/Kicad-Files/Headphone with PCM5102a and TDA1308/Kopfhoererbuchse mit PCM5102A.sch (KiCad schematic (older format))
At the start: 36 parts, among them J1 Conn_02x03_Odd_Even, J2 AudioJack3_Dual_Switch, Q1 IRLML6401, U1 PCM5102A, U2 TDA1308

Commit message: KiCad-Files umbenennen: Kopfhoererplatine
Parts:
- J2: footprint Connector_Audio:Jack_3.5mm_Cliff_Horizontal -> Kopfhoererbuchse PCM5102A:Jack_3.5mm_Cliff_Horizontal; symbol KopfhoÃàrerbuchse-mit-PCM5102A-rescue:AudioJack3_Dual_Switch-Connector -> Kopfhoererbuchse-mit-PCM5102A-rescue:AudioJack3_Dual_Switch-Connector-Kopfhörerbuchse-mit-PCM5102A
- U1: symbol KopfhoÃàrerbuchse-mit-PCM5102A-rescue:PCM5102A-Audio -> Kopfhoererbuchse-mit-PCM5102A-rescue:PCM5102A
Changed lines of the file:
@@
 encoding utf-8
 Sheet 1 1
-Title "Headphone-PCB with I2S for Tonuino"
-Date "20.04.202"
+Title "I2S-headphone-PCB for ESPuino"
+Date "2020-11-19"
 Rev ""
 Comp ""
@@
 $EndDescr
 $Comp
-L KopfhoÃàrerbuchse-mit-PCM5102A-rescue:AudioJack3_Dual_Switch-Connector J2
+L Kopfhoererbuchse-mit-PCM5102A-rescue:AudioJack3_Dual_Switch-Connector-Kopfhörerbuchse-mit-PCM5102A J2
 U 1 1 5E774924
 P 8550 4150
 F 0 "J2" H 8220 4150 50  0000 R CNN
 F 1 "AudioJack3_Dual_Switch" H 8220 4059 50  0000 R CNN
-F 2 "Connector_Audio:Jack_3.5mm_Cliff_Horizontal" H 8500 4150 50  0001 C CNN
+F 2 "Kopfhoererbuchse PCM5102A:Jack_3.5mm_Cliff_Horizontal" H 8500 4150 50  0001 C CNN
 F 3 "~" H 8500 4150 50  0001 C CNN
 	1    8550 4150
@@
 $EndComp
 $Comp
-L KopfhoÃàrerbuchse-mit-PCM5102A-rescue:PCM5102A-Audio U1
+L Kopfhoererbuchse-mit-PCM5102A-rescue:PCM5102A U1
 U 1 1 5ED93771
 P 2800 3150
