File: PCBs/Kicad-Files/Wemos Lolin32/Wemos_Lolin32.sch (KiCad schematic (older format))
At the start: 27 parts, among them J1 Neopixel, J10 RFID2, J11 Battery, J12 toLolin, J13 Reset, J2 to-Headphone, J3 RotEncoder, J4 Next-Bt, J5 RFID1, J6 Prev-Bt, J7 MAX98357a, J8 uSD-Reader, J9 PPlay-Bt, Q1 IRF530NPbF, Q2 NDP6020P, U1 Wemos Lolin32

Commit message: KiCad-Files umbenennen: Lolin32
Parts:
- C1: footprint Capacitor_THT:C_Radial_D5.0mm_H7.0mm_P2.00mm -> Capacitor_THT:CP_Radial_D4.0mm_P2.00mm
- U1: symbol symbols:Lolin32 -> Wemos_Lolin32-rescue:Lolin32-symbols
Changed lines of the file:
@@
 encoding utf-8
 Sheet 1 1
-Title "Tonuino-ESP32-I2S Lolin32"
+Title "ESPuino Lolin32"
 Date "2020-12-06"
 Rev "1.0"
@@
 NoConn ~ 5200 4150
 $Comp
-L symbols:Lolin32 U1
+L Wemos_Lolin32-rescue:Lolin32-symbols U1
 U 1 1 5F3628D0
 P 5700 3700
@@
 F 0 "C1" H 1900 2850 50  0000 L CNN
 F 1 "10uF" H 1900 2400 50  0000 L CNN
-F 2 "Capacitor_THT:C_Radial_D5.0mm_H7.0mm_P2.00mm" H 1938 2500 50  0001 C CNN
+F 2 "Capacitor_THT:CP_Radial_D4.0mm_P2.00mm" H 1938 2500 50  0001 C CNN
 F 3 "~" H 1900 2650 50  0001 C CNN
 	1    1900 2650
