File: PCBs/Kicad-Files/Wemos Lolin D32/ESPuino D32.kicad_pcb (KiCad board)
At the start: 2 copper layers, 53.3 x 81.3 mm, 21 parts, among them J1 MAX98357a, J10 uSD-Reader, J2 Neopixel, J3 to_Headphone, J4 RotEncoder, J5 Next-Bt, J6 RFID, J7 Prev-Bt, J8 PPlay-Bt, J9 Reset, M1 Lolin D32, Q1 NDP6020P, Q2 IRF530NPbF

Commit message: KiCad-Files umbenennen: Lolin D32
Other:
- board text added: "ESPuino Lolin D32 3.3V rev1.1"
- board text removed: "Tonuino Lolin D32 3.3V rev1.1"
Changed lines of the file:
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@@
-(kicad_pcb (version 20171130) (host pcbnew "(5.1.8-0-10_14)")
+(kicad_pcb (version 20171130) (host pcbnew 5.1.5+dfsg1-2build2)
   (general
     (thickness 1.6)
@@
     (uvia_dia 0.3)
     (uvia_drill 0.1)
+    (add_net +3V3)
     (add_net BUT_NEXT)
     (add_net BUT_PPLAY)
@@
     (add_net DIN)
     (add_net EN)
+    (add_net GND)
     (add_net Headphone)
     (add_net I2S_BCLK)
@@
     (uvia_dia 0.3)
     (uvia_drill 0.1)
-    (add_net +3V3)
-    (add_net GND)
   )
   (module MountingHole:MountingHole_3.2mm_M3 (layer F.Cu)
@@
   (gr_line (start 154.94 19.05) (end 154.94 100.33) (layer Edge.Cuts) (width 0.15))
   (gr_line (start 101.6 19.05) (end 154.94 19.05) (layer Edge.Cuts) (width 0.15))
-  (gr_text "Tonuino Lolin D32 3.3V rev1.1" (at 128.27 97.79) (layer B.SilkS)
+  (gr_text "ESPuino Lolin D32 3.3V rev1.1" (at 128.27 97.79) (layer B.SilkS)
     (effects (font (size 1 1) (thickness 0.15)) (justify mirror))
   )
