File: PCBs/Kicad-Files/Wemos Lolin D32/ESPuino D32.sch (KiCad schematic (older format))
At the start: 21 parts, among them J1 MAX98357a, J10 uSD-Reader, J2 Neopixel, J3 to_Headphone, J4 RotEncoder, J5 Next-Bt, J6 RFID, J7 Prev-Bt, J8 PPlay-Bt, J9 Reset, M1 LolinD32, Q1 NDP6020P, Q2 IRF530NPbF

Commit message: KiCad-Files umbenennen: Lolin D32
Parts:
- M1: symbol Tonuino-D32-rescue:LolinD32-symbols -> ESPuino-D32-rescue:LolinD32
Changed lines of the file:
@@
 $EndDescr
 $Comp
-L Tonuino-D32-rescue:LolinD32-symbols M1
+L ESPuino-D32-rescue:LolinD32 M1
 U 1 1 5FCC05A7
 P 5850 3750
