File: PCBs/Kicad-Files/Wemos Lolin32 SD_MMC PN5180/ESPuino Lolin32 MMC PN5180.kicad_pcb (KiCad board)
At the start: 2 copper layers, 55.8 x 92.7 mm, 29 parts, among them J1 to LiPo-battery, J10 Previous, J11 PPlay, J12 SD (MMC), J13 Serial, J2 to Lolin, J3 to_Headphone, J4 MAX98357a, J5 Neopixel, J6 Rotary Encoder, J7 RFID (PN5180), J8 Reset, J9 Next, Q1 IRL3103, Q2 NDP6020P, U1 Lolin32

Commit message: KiCad-Files umbenennen: Lolin32 SD_MMC PN5180
Other:
- board text added: "ESPuino Lolin32 3.3V MMC PN5180 rev1"
- board text removed: "Tonuino Lolin32 3.3V MMC PN5180 rev1"
Changed lines of the file:
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@@
-(kicad_pcb (version 20171130) (host pcbnew "(5.1.8-0-10_14)")
+(kicad_pcb (version 20171130) (host pcbnew 5.1.5+dfsg1-2build2)
   (general
     (thickness 1.6)
@@
     (effects (font (size 1.5 1.5) (thickness 0.3)))
   )
-  (gr_text "Tonuino Lolin32 3.3V MMC PN5180 rev1" (at 123.9 112.4) (layer B.SilkS)
+  (gr_text "ESPuino Lolin32 3.3V MMC PN5180 rev1" (at 123.9 112.4) (layer B.SilkS)
     (effects (font (size 1 1) (thickness 0.25)) (justify mirror))
   )
