File: PCBs/Kicad-Files/Wemos Lolin32 SD_MMC PN5180/ESPuino Lolin32 MMC PN5180.sch (KiCad schematic (older format))
At the start: 29 parts, among them J1 Battery, J10 Prev_Bt, J11 PPlay_Bt, J12 SD (MMC), J13 Serial, J2 to Lolin, J3 to_Headphone, J4 MAX98357a, J5 Neopixel, J6 Rotary Encoder, J7 RFID, J8 Reset, J9 Next_Bt, Q1 IRL3103, Q2 NDP6020P, U1 Lolin32

Commit message: KiCad-Files umbenennen: Lolin32 SD_MMC PN5180
Parts:
- U1: symbol module:Lolin32 -> ESPuino-Lolin32-MMC-PN5180-rescue:Lolin32-module
Changed lines of the file:
@@
 $EndDescr
 $Comp
-L module:Lolin32 U1
+L ESPuino-Lolin32-MMC-PN5180-rescue:Lolin32-module U1
 U 1 1 5FF660DB
 P 5550 3600
